File: placa/central/central.brd (EAGLE design)
At the start: 39 parts

Commit message: placa central
Parts:
- added IC2: 7805TV, linear:TO220V
- moved U$4 289.5 mm to (76.6, 29.7)
- moved U$8 289.4 mm to (116.8, 27.3)
- moved U$12 289.4 mm to (75.7, 60.4)
- moved JP15 289.4 mm to (27.6, 72.8)
- moved JP2 289.4 mm to (14.1, 103.7)
- moved JP24 289.4 mm to (25.9, 43.7)
- moved JP7 289.4 mm to (14.9, 72.6)
- moved JP8 289.4 mm to (13.9, 14.0)
- moved JP9 289.4 mm to (100.8, 42.6)
- moved U$1 289.4 mm to (29.6, 60.8)
- moved U$2 289.4 mm to (30.6, 120.0)
- moved U$3 289.4 mm to (77.1, 89.0)
- moved IC1 289.4 mm to (210.9, 113.9)
- moved JP1 289.4 mm to (13.2, 43.8)
- moved JP12 289.4 mm to (59.3, 43.2)
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Connections:
- net GND: now also IC2.2
- net VCC: now also IC2.3
- net VIN: now also IC2.1
Routing:
- net VCC: track 36.9 -> 1126.8 mm
- net GND: track 202.0 -> 1146.5 mm
- net N$43: track 0.00 -> 7.30 mm
- net VIN: track 73.0 -> 80.3 mm
- net N$19: track 0.00 -> 7.11 mm
- net N$21: track 0.00 -> 7.11 mm
- net N$20: track 0.00 -> 7.11 mm
- net N$45: track 0.00 -> 7.07 mm
- net N$2: track 0.00 -> 7.01 mm
- net N$38: track 0.00 -> 7.00 mm
- net N$46: track 0.00 -> 6.88 mm
- net N$3: track 0.00 -> 6.88 mm
- net N$1: track 0.00 -> 6.88 mm
- net N$26: track 0.00 -> 6.60 mm
- net N$25: track 0.00 -> 6.60 mm
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Other:
- board outline added: 220 x 135.1 mm
